File: BreadboardDAC.sch (KiCad schematic (older format))
At the start: 25 parts, among them J1 Conn_01x15

Commit message: fix footprint association for pin header
Parts:
- J1: footprint Resistor_THT:R_Axial_DIN0204_L3.6mm_D1.6mm_P7.62mm_Horizontal -> Connector_PinHeader_2.54mm:PinHeader_1x15_P2.54mm_Vertical
Changed lines of the file:
@@
 F 0 "J1" H 4018 2525 50  0000 C CNN
 F 1 "Conn_01x15" H 4018 2616 50  0000 C CNN
-F 2 "Resistor_THT:R_Axial_DIN0204_L3.6mm_D1.6mm_P7.62mm_Horizontal" H 4100 3450 50  0001 C CNN
+F 2 "Connector_PinHeader_2.54mm:PinHeader_1x15_P2.54mm_Vertical" H 4100 3450 50  0001 C CNN
 F 3 "~" H 4100 3450 50  0001 C CNN
 	1    4100 3450

Commit message: use vertical orientation for resistors
Parts:
- R1, R10, R11, R12, R13, R14, R15, R16, R17, R18, R19, R2, R20, R21, R22, R23, R24, R3, R4, R5, R6, R7, R8, R9: footprint Resistor_THT:R_Axial_DIN0204_L3.6mm_D1.6mm_P7.62mm_Horizontal -> Resistor_THT:R_Axial_DIN0204_L3.6mm_D1.6mm_P2.54mm_Vertical
Changed lines of the file:
@@
 F 0 "R9" V 4900 4050 50  0000 C CNN
 F 1 "3k9" V 4950 3850 50  0000 C CNN
-F 2 "Resistor_THT:R_Axial_DIN0204_L3.6mm_D1.6mm_P7.62mm_Horizontal" V 4880 3850 50  0001 C CNN
+F 2 "Resistor_THT:R_Axial_DIN0204_L3.6mm_D1.6mm_P2.54mm_Vertical" V 4880 3850 50  0001 C CNN
 F 3 "" H 4950 3850 50  0001 C CNN
 	1    4950 3850
@@
 F 0 "R21" V 5400 4050 50  0000 C CNN
 F 1 "200" V 5450 3850 50  0000 C CNN
-F 2 "Resistor_THT:R_Axial_DIN0204_L3.6mm_D1.6mm_P7.62mm_Horizontal" V 5380 3850 50  0001 C CNN
+F 2 "Resistor_THT:R_Axial_DIN0204_L3.6mm_D1.6mm_P2.54mm_Vertical" V 5380 3850 50  0001 C CNN
 F 3 "" H 5450 3850 50  0001 C CNN
 	1    5450 3850
@@
 F 0 "R10" V 4900 4150 50  0000 C CNN
 F 1 "2k" V 4950 3950 50  0000 C CNN
-F 2 "Resistor_THT:R_Axial_DIN0204_L3.6mm_D1.6mm_P7.62mm_Horizontal" V 4880 3950 50  0001 C CNN
+F 2 "Resistor_THT:R_Axial_DIN0204_L3.6mm_D1.6mm_P2.54mm_Vertical" V 4880 3950 50  0001 C CNN
 F 3 "" H 4950 3950 50  0001 C CNN
 	1    4950 3950
@@
 F 0 "R22" V 5400 4150 50  0000 C CNN
 F 1 "51" V 5450 3950 50  0000 C CNN
-F 2 "Resistor_THT:R_Axial_DIN0204_L3.6mm_D1.6mm_P7.62mm_Horizontal" V 5380 3950 50  0001 C CNN
+F 2 "Resistor_THT:R_Axial_DIN0204_L3.6mm_D1.6mm_P2.54mm_Vertical" V 5380 3950 50  0001 C CNN
 F 3 "" H 5450 3950 50  0001 C CNN
 	1    5450 3950
@@
 F 0 "R11" V 4900 4250 50  0000 C CNN
 F 1 "1k" V 4950 4050 50  0000 C CNN
-F 2 "Resistor_THT:R_Axial_DIN0204_L3.6mm_D1.6mm_P7.62mm_Horizontal" V 4880 4050 50  0001 C CNN
+F 2 "Resistor_THT:R_Axial_DIN0204_L3.6mm_D1.6mm_P2.54mm_Vertical" V 4880 4050 50  0001 C CNN
 F 3 "" H 4950 4050 50  0001 C CNN
 	1    4950 4050
@@
 F 0 "R23" V 5400 4250 50  0000 C CNN
 F 1 "24" V 5450 4050 50  0000 C CNN
-F 2 "Resistor_THT:R_Axial_DIN0204_L3.6mm_D1.6mm_P7.62mm_Horizontal" V 5380 4050 50  0001 C CNN
+F 2 "Resistor_THT:R_Axial_DIN0204_L3.6mm_D1.6mm_P2.54mm_Vertical" V 5380 4050 50  0001 C CNN
 F 3 "" H 5450 4050 50  0001 C CNN
 	1    5450 4050
@@
 F 0 "R12" V 4900 4350 50  0000 C CNN
 F 1 "430" V 4950 4150 50  0000 C CNN
-F 2 "Resistor_THT:R_Axial_DIN0204_L3.6mm_D1.6mm_P7.62mm_Horizontal" V 4880 4150 50  0001 C CNN
+F 2 "Resistor_THT:R_Axial_DIN0204_L3.6mm_D1.6mm_P2.54mm_Vertical" V 4880 4150 50  0001 C CNN
 F 3 "" H 4950 4150 50  0001 C CNN
 	1    4950 4150
@@
 F 0 "R24" V 5400 4350 50  0000 C CNN
 F 1 "82" V 5450 4150 50  0000 C CNN
-F 2 "Resistor_THT:R_Axial_DIN0204_L3.6mm_D1.6mm_P7.62mm_Horizontal" V 5380 4150 50  0001 C CNN
+F 2 "Resistor_THT:R_Axial_DIN0204_L3.6mm_D1.6mm_P2.54mm_Vertical" V 5380 4150 50  0001 C CNN
 F 3 "" H 5450 4150 50  0001 C CNN
 	1    5450 4150
@@
 F 0 "R5" V 4900 3650 50  0000 C CNN
 F 1 "3k9" V 4950 3450 50  0000 C CNN
-F 2 "Resistor_THT:R_Axial_DIN0204_L3.6mm_D1.6mm_P7.62mm_Horizontal" V 4880 3450 50  0001 C CNN
+F 2 "Resistor_THT:R_Axial_DIN0204_L3.6mm_D1.6mm_P2.54mm_Vertical" V 4880 3450 50  0001 C CNN
 F 3 "" H 4950 3450 50  0001 C CNN
 	1    4950 3450
@@
 F 0 "R17" V 5400 3650 50  0000 C CNN
 F 1 "200" V 5450 3450 50  0000 C CNN
-F 2 "Resistor_THT:R_Axial_DIN0204_L3.6mm_D1.6mm_P7.62mm_Horizontal" V 5380 3450 50  0001 C CNN
+F 2 "Resistor_THT:R_Axial_DIN0204_L3.6mm_D1.6mm_P2.54mm_Vertical" V 5380 3450 50  0001 C CNN
 F 3 "" H 5450 3450 50  0001 C CNN
 	1    5450 3450
@@
 F 0 "R6" V 4900 3750 50  0000 C CNN
 F 1 "2k" V 4950 3550 50  0000 C CNN
-F 2 "Resistor_THT:R_Axial_DIN0204_L3.6mm_D1.6mm_P7.62mm_Horizontal" V 4880 3550 50  0001 C CNN
+F 2 "Resistor_THT:R_Axial_DIN0204_L3.6mm_D1.6mm_P2.54mm_Vertical" V 4880 3550 50  0001 C CNN
 F 3 "" H 4950 3550 50  0001 C CNN
 	1    4950 3550
@@
 F 0 "R18" V 5400 3750 50  0000 C CNN
 F 1 "51" V 5450 3550 50  0000 C CNN
-F 2 "Resistor_THT:R_Axial_DIN0204_L3.6mm_D1.6mm_P7.62mm_Horizontal" V 5380 3550 50  0001 C CNN
+F 2 "Resistor_THT:R_Axial_DIN0204_L3.6mm_D1.6mm_P2.54mm_Vertical" V 5380 3550 50  0001 C CNN
 F 3 "" H 5450 3550 50  0001 C CNN
 	1    5450 3550
@@
 F 0 "R7" V 4900 3850 50  0000 C CNN
 F 1 "1k" V 4950 3650 50  0000 C CNN
-F 2 "Resistor_THT:R_Axial_DIN0204_L3.6mm_D1.6mm_P7.62mm_Horizontal" V 4880 3650 50  0001 C CNN
+F 2 "Resistor_THT:R_Axial_DIN0204_L3.6mm_D1.6mm_P2.54mm_Vertical" V 4880 3650 50  0001 C CNN
 F 3 "" H 4950 3650 50  0001 C CNN
 	1    4950 3650
@@
 F 0 "R19" V 5400 3850 50  0000 C CNN
 F 1 "24" V 5450 3650 50  0000 C CNN
-F 2 "Resistor_THT:R_Axial_DIN0204_L3.6mm_D1.6mm_P7.62mm_Horizontal" V 5380 3650 50  0001 C CNN
+F 2 "Resistor_THT:R_Axial_DIN0204_L3.6mm_D1.6mm_P2.54mm_Vertical" V 5380 3650 50  0001 C CNN
 F 3 "" H 5450 3650 50  0001 C CNN
 	1    5450 3650
@@
 F 0 "R8" V 4900 3950 50  0000 C CNN
 F 1 "430" V 4950 3750 50  0000 C CNN
-F 2 "Resistor_THT:R_Axial_DIN0204_L3.6mm_D1.6mm_P7.62mm_Horizontal" V 4880 3750 50  0001 C CNN
+F 2 "Resistor_THT:R_Axial_DIN0204_L3.6mm_D1.6mm_P2.54mm_Vertical" V 4880 3750 50  0001 C CNN
 F 3 "" H 4950 3750 50  0001 C CNN
 	1    4950 3750
@@
 F 0 "R20" V 5400 3950 50  0000 C CNN
 F 1 "82" V 5450 3750 50  0000 C CNN
-F 2 "Resistor_THT:R_Axial_DIN0204_L3.6mm_D1.6mm_P7.62mm_Horizontal" V 5380 3750 50  0001 C CNN
+F 2 "Resistor_THT:R_Axial_DIN0204_L3.6mm_D1.6mm_P2.54mm_Vertical" V 5380 3750 50  0001 C CNN
 F 3 "" H 5450 3750 50  0001 C CNN
 	1    5450 3750
@@
 F 0 "R1" V 4900 3250 50  0000 C CNN
 F 1 "3k9" V 4950 3050 50  0000 C CNN
-F 2 "Resistor_THT:R_Axial_DIN0204_L3.6mm_D1.6mm_P7.62mm_Horizontal" V 4880 3050 50  0001 C CNN
+F 2 "Resistor_THT:R_Axial_DIN0204_L3.6mm_D1.6mm_P2.54mm_Vertical" V 4880 3050 50  0001 C CNN
 F 3 "" H 4950 3050 50  0001 C CNN
 	1    4950 3050
@@
 F 0 "R13" V 5400 3250 50  0000 C CNN
 F 1 "200" V 5450 3050 50  0000 C CNN
-F 2 "Resistor_THT:R_Axial_DIN0204_L3.6mm_D1.6mm_P7.62mm_Horizontal" V 5380 3050 50  0001 C CNN
+F 2 "Resistor_THT:R_Axial_DIN0204_L3.6mm_D1.6mm_P2.54mm_Vertical" V 5380 3050 50  0001 C CNN
 F 3 "" H 5450 3050 50  0001 C CNN
 	1    5450 3050
@@
 F 0 "R2" V 4900 3350 50  0000 C CNN
 F 1 "2k" V 4950 3150 50  0000 C CNN
-F 2 "Resistor_THT:R_Axial_DIN0204_L3.6mm_D1.6mm_P7.62mm_Horizontal" V 4880 3150 50  0001 C CNN
+F 2 "Resistor_THT:R_Axial_DIN0204_L3.6mm_D1.6mm_P2.54mm_Vertical" V 4880 3150 50  0001 C CNN
 F 3 "" H 4950 3150 50  0001 C CNN
 	1    4950 3150
@@
 F 0 "R14" V 5400 3350 50  0000 C CNN
 F 1 "51" V 5450 3150 50  0000 C CNN
-F 2 "Resistor_THT:R_Axial_DIN0204_L3.6mm_D1.6mm_P7.62mm_Horizontal" V 5380 3150 50  0001 C CNN
+F 2 "Resistor_THT:R_Axial_DIN0204_L3.6mm_D1.6mm_P2.54mm_Vertical" V 5380 3150 50  0001 C CNN
 F 3 "" H 5450 3150 50  0001 C CNN
 	1    5450 3150
@@
 F 0 "R3" V 4900 3450 50  0000 C CNN
 F 1 "1k" V 4950 3250 50  0000 C CNN
-F 2 "Resistor_THT:R_Axial_DIN0204_L3.6mm_D1.6mm_P7.62mm_Horizontal" V 4880 3250 50  0001 C CNN
+F 2 "Resistor_THT:R_Axial_DIN0204_L3.6mm_D1.6mm_P2.54mm_Vertical" V 4880 3250 50  0001 C CNN
 F 3 "" H 4950 3250 50  0001 C CNN
 	1    4950 3250
@@
 F 0 "R15" V 5400 3450 50  0000 C CNN
 F 1 "24" V 5450 3250 50  0000 C CNN
-F 2 "Resistor_THT:R_Axial_DIN0204_L3.6mm_D1.6mm_P7.62mm_Horizontal" V 5380 3250 50  0001 C CNN
+F 2 "Resistor_THT:R_Axial_DIN0204_L3.6mm_D1.6mm_P2.54mm_Vertical" V 5380 3250 50  0001 C CNN
 F 3 "" H 5450 3250 50  0001 C CNN
 	1    5450 3250
@@
 F 0 "R4" V 4900 3550 50  0000 C CNN
 F 1 "430" V 4950 3350 50  0000 C CNN
-F 2 "Resistor_THT:R_Axial_DIN0204_L3.6mm_D1.6mm_P7.62mm_Horizontal" V 4880 3350 50  0001 C CNN
+F 2 "Resistor_THT:R_Axial_DIN0204_L3.6mm_D1.6mm_P2.54mm_Vertical" V 4880 3350 50  0001 C CNN
 F 3 "" H 4950 3350 50  0001 C CNN
 	1    4950 3350
@@
 F 0 "R16" V 5400 3550 50  0000 C CNN
 F 1 "82" V 5450 3350 50  0000 C CNN
-F 2 "Resistor_THT:R_Axial_DIN0204_L3.6mm_D1.6mm_P7.62mm_Horizontal" V 5380 3350 50  0001 C CNN
+F 2 "Resistor_THT:R_Axial_DIN0204_L3.6mm_D1.6mm_P2.54mm_Vertical" V 5380 3350 50  0001 C CNN
 F 3 "" H 5450 3350 50  0001 C CNN
 	1    5450 3350

Commit message: completed design?
Parts:
- R1, R10, R11, R12, R13, R14, R15, R16, R17, R18, R19, R2, R20, R21, R22, R23, R24, R3, R4, R5, R6, R7, R8, R9: footprint Resistor_THT:R_Axial_DIN0204_L3.6mm_D1.6mm_P2.54mm_Vertical -> BreadboardDAC:R_Axial_DIN0204_L3.6mm_D1.6mm_P2.54mm_Vertical
Changed lines of the file:
@@
 F 0 "R9" V 4900 4050 50  0000 C CNN
 F 1 "3k9" V 4950 3850 50  0000 C CNN
-F 2 "Resistor_THT:R_Axial_DIN0204_L3.6mm_D1.6mm_P2.54mm_Vertical" V 4880 3850 50  0001 C CNN
+F 2 "BreadboardDAC:R_Axial_DIN0204_L3.6mm_D1.6mm_P2.54mm_Vertical" V 4880 3850 50  0001 C CNN
 F 3 "" H 4950 3850 50  0001 C CNN
 	1    4950 3850
@@
 F 0 "R21" V 5400 4050 50  0000 C CNN
 F 1 "200" V 5450 3850 50  0000 C CNN
-F 2 "Resistor_THT:R_Axial_DIN0204_L3.6mm_D1.6mm_P2.54mm_Vertical" V 5380 3850 50  0001 C CNN
+F 2 "BreadboardDAC:R_Axial_DIN0204_L3.6mm_D1.6mm_P2.54mm_Vertical" V 5380 3850 50  0001 C CNN
 F 3 "" H 5450 3850 50  0001 C CNN
 	1    5450 3850
@@
 F 0 "R10" V 4900 4150 50  0000 C CNN
 F 1 "2k" V 4950 3950 50  0000 C CNN
-F 2 "Resistor_THT:R_Axial_DIN0204_L3.6mm_D1.6mm_P2.54mm_Vertical" V 4880 3950 50  0001 C CNN
+F 2 "BreadboardDAC:R_Axial_DIN0204_L3.6mm_D1.6mm_P2.54mm_Vertical" V 4880 3950 50  0001 C CNN
 F 3 "" H 4950 3950 50  0001 C CNN
 	1    4950 3950
@@
 F 0 "R22" V 5400 4150 50  0000 C CNN
 F 1 "51" V 5450 3950 50  0000 C CNN
-F 2 "Resistor_THT:R_Axial_DIN0204_L3.6mm_D1.6mm_P2.54mm_Vertical" V 5380 3950 50  0001 C CNN
+F 2 "BreadboardDAC:R_Axial_DIN0204_L3.6mm_D1.6mm_P2.54mm_Vertical" V 5380 3950 50  0001 C CNN
 F 3 "" H 5450 3950 50  0001 C CNN
 	1    5450 3950
@@
 F 0 "R11" V 4900 4250 50  0000 C CNN
 F 1 "1k" V 4950 4050 50  0000 C CNN
-F 2 "Resistor_THT:R_Axial_DIN0204_L3.6mm_D1.6mm_P2.54mm_Vertical" V 4880 4050 50  0001 C CNN
+F 2 "BreadboardDAC:R_Axial_DIN0204_L3.6mm_D1.6mm_P2.54mm_Vertical" V 4880 4050 50  0001 C CNN
 F 3 "" H 4950 4050 50  0001 C CNN
 	1    4950 4050
@@
 F 0 "R23" V 5400 4250 50  0000 C CNN
 F 1 "24" V 5450 4050 50  0000 C CNN
-F 2 "Resistor_THT:R_Axial_DIN0204_L3.6mm_D1.6mm_P2.54mm_Vertical" V 5380 4050 50  0001 C CNN
+F 2 "BreadboardDAC:R_Axial_DIN0204_L3.6mm_D1.6mm_P2.54mm_Vertical" V 5380 4050 50  0001 C CNN
 F 3 "" H 5450 4050 50  0001 C CNN
 	1    5450 4050
@@
 F 0 "R12" V 4900 4350 50  0000 C CNN
 F 1 "430" V 4950 4150 50  0000 C CNN
-F 2 "Resistor_THT:R_Axial_DIN0204_L3.6mm_D1.6mm_P2.54mm_Vertical" V 4880 4150 50  0001 C CNN
+F 2 "BreadboardDAC:R_Axial_DIN0204_L3.6mm_D1.6mm_P2.54mm_Vertical" V 4880 4150 50  0001 C CNN
 F 3 "" H 4950 4150 50  0001 C CNN
 	1    4950 4150
@@
 F 0 "R24" V 5400 4350 50  0000 C CNN
 F 1 "82" V 5450 4150 50  0000 C CNN
-F 2 "Resistor_THT:R_Axial_DIN0204_L3.6mm_D1.6mm_P2.54mm_Vertical" V 5380 4150 50  0001 C CNN
+F 2 "BreadboardDAC:R_Axial_DIN0204_L3.6mm_D1.6mm_P2.54mm_Vertical" V 5380 4150 50  0001 C CNN
 F 3 "" H 5450 4150 50  0001 C CNN
 	1    5450 4150
@@
 F 0 "R5" V 4900 3650 50  0000 C CNN
 F 1 "3k9" V 4950 3450 50  0000 C CNN
-F 2 "Resistor_THT:R_Axial_DIN0204_L3.6mm_D1.6mm_P2.54mm_Vertical" V 4880 3450 50  0001 C CNN
+F 2 "BreadboardDAC:R_Axial_DIN0204_L3.6mm_D1.6mm_P2.54mm_Vertical" V 4880 3450 50  0001 C CNN
 F 3 "" H 4950 3450 50  0001 C CNN
 	1    4950 3450
@@
 F 0 "R17" V 5400 3650 50  0000 C CNN
 F 1 "200" V 5450 3450 50  0000 C CNN
-F 2 "Resistor_THT:R_Axial_DIN0204_L3.6mm_D1.6mm_P2.54mm_Vertical" V 5380 3450 50  0001 C CNN
+F 2 "BreadboardDAC:R_Axial_DIN0204_L3.6mm_D1.6mm_P2.54mm_Vertical" V 5380 3450 50  0001 C CNN
 F 3 "" H 5450 3450 50  0001 C CNN
 	1    5450 3450
@@
 F 0 "R6" V 4900 3750 50  0000 C CNN
 F 1 "2k" V 4950 3550 50  0000 C CNN
-F 2 "Resistor_THT:R_Axial_DIN0204_L3.6mm_D1.6mm_P2.54mm_Vertical" V 4880 3550 50  0001 C CNN
+F 2 "BreadboardDAC:R_Axial_DIN0204_L3.6mm_D1.6mm_P2.54mm_Vertical" V 4880 3550 50  0001 C CNN
 F 3 "" H 4950 3550 50  0001 C CNN
 	1    4950 3550
@@
 F 0 "R18" V 5400 3750 50  0000 C CNN
 F 1 "51" V 5450 3550 50  0000 C CNN
-F 2 "Resistor_THT:R_Axial_DIN0204_L3.6mm_D1.6mm_P2.54mm_Vertical" V 5380 3550 50  0001 C CNN
+F 2 "BreadboardDAC:R_Axial_DIN0204_L3.6mm_D1.6mm_P2.54mm_Vertical" V 5380 3550 50  0001 C CNN
 F 3 "" H 5450 3550 50  0001 C CNN
 	1    5450 3550
@@
 F 0 "R7" V 4900 3850 50  0000 C CNN
 F 1 "1k" V 4950 3650 50  0000 C CNN
-F 2 "Resistor_THT:R_Axial_DIN0204_L3.6mm_D1.6mm_P2.54mm_Vertical" V 4880 3650 50  0001 C CNN
+F 2 "BreadboardDAC:R_Axial_DIN0204_L3.6mm_D1.6mm_P2.54mm_Vertical" V 4880 3650 50  0001 C CNN
 F 3 "" H 4950 3650 50  0001 C CNN
 	1    4950 3650
@@
 F 0 "R19" V 5400 3850 50  0000 C CNN
 F 1 "24" V 5450 3650 50  0000 C CNN
-F 2 "Resistor_THT:R_Axial_DIN0204_L3.6mm_D1.6mm_P2.54mm_Vertical" V 5380 3650 50  0001 C CNN
+F 2 "BreadboardDAC:R_Axial_DIN0204_L3.6mm_D1.6mm_P2.54mm_Vertical" V 5380 3650 50  0001 C CNN
 F 3 "" H 5450 3650 50  0001 C CNN
 	1    5450 3650
@@
 F 0 "R8" V 4900 3950 50  0000 C CNN
 F 1 "430" V 4950 3750 50  0000 C CNN
-F 2 "Resistor_THT:R_Axial_DIN0204_L3.6mm_D1.6mm_P2.54mm_Vertical" V 4880 3750 50  0001 C CNN
+F 2 "BreadboardDAC:R_Axial_DIN0204_L3.6mm_D1.6mm_P2.54mm_Vertical" V 4880 3750 50  0001 C CNN
 F 3 "" H 4950 3750 50  0001 C CNN
 	1    4950 3750
@@
 F 0 "R20" V 5400 3950 50  0000 C CNN
 F 1 "82" V 5450 3750 50  0000 C CNN
-F 2 "Resistor_THT:R_Axial_DIN0204_L3.6mm_D1.6mm_P2.54mm_Vertical" V 5380 3750 50  0001 C CNN
+F 2 "BreadboardDAC:R_Axial_DIN0204_L3.6mm_D1.6mm_P2.54mm_Vertical" V 5380 3750 50  0001 C CNN
 F 3 "" H 5450 3750 50  0001 C CNN
 	1    5450 3750
@@
 F 0 "R1" V 4900 3250 50  0000 C CNN
 F 1 "3k9" V 4950 3050 50  0000 C CNN
-F 2 "Resistor_THT:R_Axial_DIN0204_L3.6mm_D1.6mm_P2.54mm_Vertical" V 4880 3050 50  0001 C CNN
+F 2 "BreadboardDAC:R_Axial_DIN0204_L3.6mm_D1.6mm_P2.54mm_Vertical" V 4880 3050 50  0001 C CNN
 F 3 "" H 4950 3050 50  0001 C CNN
 	1    4950 3050
@@
 F 0 "R13" V 5400 3250 50  0000 C CNN
 F 1 "200" V 5450 3050 50  0000 C CNN
-F 2 "Resistor_THT:R_Axial_DIN0204_L3.6mm_D1.6mm_P2.54mm_Vertical" V 5380 3050 50  0001 C CNN
+F 2 "BreadboardDAC:R_Axial_DIN0204_L3.6mm_D1.6mm_P2.54mm_Vertical" V 5380 3050 50  0001 C CNN
 F 3 "" H 5450 3050 50  0001 C CNN
 	1    5450 3050
@@
 F 0 "R2" V 4900 3350 50  0000 C CNN
 F 1 "2k" V 4950 3150 50  0000 C CNN
-F 2 "Resistor_THT:R_Axial_DIN0204_L3.6mm_D1.6mm_P2.54mm_Vertical" V 4880 3150 50  0001 C CNN
+F 2 "BreadboardDAC:R_Axial_DIN0204_L3.6mm_D1.6mm_P2.54mm_Vertical" V 4880 3150 50  0001 C CNN
 F 3 "" H 4950 3150 50  0001 C CNN
 	1    4950 3150
@@
 F 0 "R14" V 5400 3350 50  0000 C CNN
 F 1 "51" V 5450 3150 50  0000 C CNN
-F 2 "Resistor_THT:R_Axial_DIN0204_L3.6mm_D1.6mm_P2.54mm_Vertical" V 5380 3150 50  0001 C CNN
+F 2 "BreadboardDAC:R_Axial_DIN0204_L3.6mm_D1.6mm_P2.54mm_Vertical" V 5380 3150 50  0001 C CNN
 F 3 "" H 5450 3150 50  0001 C CNN
 	1    5450 3150
@@
 F 0 "R3" V 4900 3450 50  0000 C CNN
 F 1 "1k" V 4950 3250 50  0000 C CNN
-F 2 "Resistor_THT:R_Axial_DIN0204_L3.6mm_D1.6mm_P2.54mm_Vertical" V 4880 3250 50  0001 C CNN
+F 2 "BreadboardDAC:R_Axial_DIN0204_L3.6mm_D1.6mm_P2.54mm_Vertical" V 4880 3250 50  0001 C CNN
 F 3 "" H 4950 3250 50  0001 C CNN
 	1    4950 3250
@@
 F 0 "R15" V 5400 3450 50  0000 C CNN
 F 1 "24" V 5450 3250 50  0000 C CNN
-F 2 "Resistor_THT:R_Axial_DIN0204_L3.6mm_D1.6mm_P2.54mm_Vertical" V 5380 3250 50  0001 C CNN
+F 2 "BreadboardDAC:R_Axial_DIN0204_L3.6mm_D1.6mm_P2.54mm_Vertical" V 5380 3250 50  0001 C CNN
 F 3 "" H 5450 3250 50  0001 C CNN
 	1    5450 3250
@@
 F 0 "R4" V 4900 3550 50  0000 C CNN
 F 1 "430" V 4950 3350 50  0000 C CNN
-F 2 "Resistor_THT:R_Axial_DIN0204_L3.6mm_D1.6mm_P2.54mm_Vertical" V 4880 3350 50  0001 C CNN
+F 2 "BreadboardDAC:R_Axial_DIN0204_L3.6mm_D1.6mm_P2.54mm_Vertical" V 4880 3350 50  0001 C CNN
 F 3 "" H 4950 3350 50  0001 C CNN
 	1    4950 3350
@@
 F 0 "R16" V 5400 3550 50  0000 C CNN
 F 1 "82" V 5450 3350 50  0000 C CNN
-F 2 "Resistor_THT:R_Axial_DIN0204_L3.6mm_D1.6mm_P2.54mm_Vertical" V 5380 3350 50  0001 C CNN
+F 2 "BreadboardDAC:R_Axial_DIN0204_L3.6mm_D1.6mm_P2.54mm_Vertical" V 5380 3350 50  0001 C CNN
 F 3 "" H 5450 3350 50  0001 C CNN
 	1    5450 3350
